File: sensor_board.sch (KiCad schematic (older format))
At the start: 5 parts, among them J1 Sensor0, J2 Sensor1

Commit message: made it teensy
Parts:
- removed A1: Arduino_UNO_R3, Module:Arduino_UNO_R3, symbol MCU_Module:Arduino_UNO_R3
- added J3: iBUS-RX, Connector_PinHeader_2.54mm:PinHeader_1x03_P2.54mm_Horizontal, symbol Connector_Generic:Conn_01x03
- added J4: iBUS-TX, Connector_PinHeader_2.54mm:PinHeader_1x03_P2.54mm_Horizontal, symbol Connector_Generic:Conn_01x03
- added J5: teensyLeft, Connector_PinSocket_2.54mm:PinSocket_1x14_P2.54mm_Vertical, symbol Connector_Generic:Conn_01x14
- added J6: teensyRight, Connector_PinSocket_2.54mm:PinSocket_1x14_P2.54mm_Vertical, symbol Connector_Generic:Conn_01x14
- added R1: 11k5, Resistor_SMD:R_0603_1608Metric_Pad1.05x0.95mm_HandSolder, symbol Device:R_Small
- added R2: 22k1, Resistor_SMD:R_0603_1608Metric_Pad1.05x0.95mm_HandSolder, symbol Device:R_Small
Connections:
- net +5V: now also J3.3 (Pin_3), J4.3 (Pin_3), J6.1 (Pin_1); no longer C1.1, C2.1, J1.6 (Pin_6), J2.6 (Pin_6)
- net GND: now also J3.1 (Pin_1), J4.1 (Pin_1), J5.1 (Pin_1), J6.2 (Pin_2), R2.2
- net GPIO_0: now also J6.12 (Pin_12)
- net GPIO_1: now also J6.10 (Pin_10)
- net SCL: now also J6.8 (Pin_8)
- net SDA: now also J6.9 (Pin_9)
- net ~XSHUT_0: now also J6.13 (Pin_13)
- net ~XSHUT_1: now also J6.11 (Pin_11)
- new net: J3.2 (Pin_2), R1.1
- new net +3V3: C1.1, C2.1, J1.6 (Pin_6), J2.6 (Pin_6), J6.3 (Pin_3)
- new net iBUS-RX: J5.11 (Pin_11), R1.2, R2.1
- new net iBUS-TX: J4.2 (Pin_2), J5.12 (Pin_12)
Other:
- moved on the sheet: C1, C2, J1, J2
